File: Relay_Board_V3.1.brd (EAGLE design)
At the start: 140 x 100 mm, 53 parts

Commit message: Major Trace Routes
Parts:
- moved U$22 1.00 mm to (62.0, 14.0), flipped to the bottom, turned to 90 degrees
Routing:
- added copper zone on layer 1, net CAP_FUSE
- added copper zone on layer 1, net CAP_SENSOR
- added copper zone on layer 1, net CHARGING_RES_NEG
- added copper zone on layer 1, net FC_POS
- added copper zone on layer 16, net FC_POS
- added copper zone on layer 1, net FC_POWER
- added copper zone on layer 1, net FC_SENSOR
- added copper zone on layer 1, net GND
- added copper zone on layer 1, net MOTOR_C_SENSOR
- added copper zone on layer 1, net MOTOR_POS

Commit message: Board Routed
Parts:
- added R14, R15, R16: 1.5k (0.1%), Resistor:R0805
- added S1, S2, S3: (no value), SparkFun-Electromechanical:SWITCH-SPDT
- R2, R4: value 750(<1%) -> 775 (0.1%)
- R5, R8: value 9250 (<1%) -> 10.5k (0.1%)
- R6: value 9250(1%) -> 10.5k (0.1%)
- R7: value 750(1%) -> 775 (0.1%)
- moved C2 89.4 mm to (49.5, 67.0), turned to 90 degrees
- moved C3 78.2 mm to (60.0, 33.0), turned to 180 degrees
- moved U$16 69.5 mm to (61.5, 27.0), turned to 180 degrees
- moved U$15 58.2 mm to (132.5, 25.5), turned to 180 degrees
- moved R2 39.7 mm to (72.0, 59.5)
- moved R3 28.3 mm to (135.0, 86.0)
- moved C1 27.7 mm to (112.5, 45.5), turned to 0 degrees
- moved R12 22.8 mm to (135.0, 67.0), turned to 270 degrees
- moved R18 22.3 mm to (135.0, 76.5), turned to 270 degrees
- moved R1 19.9 mm to (120.0, 81.5), turned to 180 degrees
- moved R13 17.5 mm to (120.0, 72.0)
- moved R6 16.4 mm to (18.0, 73.0), turned to 0 degrees
- moved U$11 12.7 mm to (120.0, 78.5), turned to 270 degrees
- moved R5 11.9 mm to (122.5, 21.0)
- moved U$6 11.7 mm to (128.0, 65.5)
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- renumbered U$10 to D1
Connections:
- new net N$10: R14.1, S1.3
- new net N$11: R2.1, S3.1
- new net N$12: R15.1, S3.3
- new net N$16: R7.1, S2.1
- new net N$17: R16.1, S2.3
- new net N$9: R4.1, S1.1
- net CAP_SENSOR: now also U$13.NO(++)
- net CAP_VOLT: now also S1.2; no longer R4.2
- net FC_POS: now also U$13.NO(--)
- net FC_VOLT: now also S2.2; no longer R7.2
- net GND: now also R14.2, R15.2, R16.2, R2.2, R4.2, R7.2, U$13.(--), U$14.(--); no longer R2.1, R4.1, R7.1
- net MOTOR_C_SENSOR: now also U$14.NO(--)
- net MOTOR_POS: now also U$14.NO(++)
- net MOTOR_VOLT: now also S3.2; no longer R2.2
- net N$13: now also U$13.(++)
- net N$6: now also U$14.(++)
Routing:
- net GND: track 0.00 -> 447.2 mm, vias 0 -> 3
- net ISO_GND: track 0.00 -> 250.2 mm
- net 5V: track 0.00 -> 231.8 mm, vias 0 -> 3
- net FC_VOLT: track 0.00 -> 166.5 mm, vias 0 -> 3
- net MOTOR_R: track 0.00 -> 155.3 mm
- net FC_CURR: track 0.00 -> 149.7 mm, vias 0 -> 1
- net FC.12: track 0.00 -> 119.5 mm
- net CHARGE_R: track 0.00 -> 115.8 mm
- net MOTOR_VOLT: track 0.00 -> 109.7 mm, vias 0 -> 1
- net N$30: track 0.00 -> 97.6 mm
- net START_R: track 0.00 -> 92.1 mm
- net POWER_BOARD: track 0.00 -> 91.1 mm
- net AUX.12: track 0.00 -> 85.6 mm
- net FCC_R: track 0.00 -> 82.1 mm, vias 0 -> 1
- net CAP_R: track 0.00 -> 79.2 mm
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- removed copper zone on layer 16, net FC_POS
