File: Relay_Board_V3.1.sch (EAGLE design)
At the start: 50 parts

Commit message: Schematic Complete
Parts:
- removed START.RELAY3, START.RELAY4: VCF4-1000, VCF4-1000:VCF4-1000
- added U$10: APT60S20SG, Diode - APT60S20SG:APT60S20SG
- added U$13, U$14: 255-5246-ND, Relay 255-5246-ND:255-5246-ND
- added U$15, U$16: P6KE15A-E3/54GICT-ND_TVS_DIODE, TVS Diode Through-Hole:P6KE15A-E3/54GICT-ND_TVS_DIODE
- R2, R4, R5, R6, R7, R8: device resistor:R-US_R0805 -> Resistor:R-US_R0805
Connections:
- removed net POWER_IN: FC.POS.P$1
- net AUX.12: now also U$16.P(-)
- net CAP_FUSE: no longer START.RELAY2.30, START.RELAY4.30
- net CAP_SENSOR: now also START.RELAY2.30, U$13.N.O.(+)
- net FC.12: now also U$15.P(-)
- net FC_POS: now also U$10.(-), U$13.N.O.(-); no longer START.RELAY4.87
- net FC_POWER: now also U$10.(+)
- net FC_SENSOR: now also FC.POS.P$1
- net GND: now also U$13.(-), U$14.(-), U$15.P(+), U$16.P(+); no longer START.RELAY3.85, START.RELAY4.85
- net MOTOR_C_SENSOR: now also U$14.N.O.(-); no longer START.RELAY3.87
- net MOTOR_POS: now also U$14.N.O.(+); no longer START.RELAY3.30
- net N$13: now also U$13.(+); no longer START.RELAY4.86
- net N$6: now also U$14.(+); no longer START.RELAY3.86
Other:
- note removed: "(INSERT DIODE HERE)"

Commit message: Board Routed
Parts:
- added R14, R15, R16: 1.5k (0.1%), Resistor:R-US_R0805
- added S1, S2, S3: (no value), SparkFun-Electromechanical:SWITCH-SPDTPTH
- R2, R4: value 750(<1%) -> 775 (0.1%)
- R5, R8: value 9250 (<1%) -> 10.5k (0.1%)
- R6: value 9250(1%) -> 10.5k (0.1%)
- R7: value 750(1%) -> 775 (0.1%)
- renumbered U$10 to D1
Connections:
- new net N$10: R14.1, S1.S
- new net N$11: R2.1, S3.O
- new net N$12: R15.1, S3.S
- new net N$16: R7.1, S2.O
- new net N$17: R16.1, S2.S
- new net N$9: R4.1, S1.O
- net CAP_VOLT: now also S1.P; no longer R4.2
- net FC_VOLT: now also S2.P; no longer R7.2
- net GND: now also R14.2, R15.2, R16.2, R2.2, R4.2, R7.2; no longer R2.1, R4.1, R7.1
- net MOTOR_VOLT: now also S3.P; no longer R2.2
Other:
- moved on the sheet: R2, R4, R5, R6, R7, R8
