File: Relay_Board_V3.2.sch (EAGLE design)
At the start: 59 parts

Commit message: Updated OptoIsolator Part so it is same as FCC
Parts:
- R14, R15, R16, R2, R4, R5, R6, R7, R8: device Resistor:R-US_R0805 -> resistor:R-US_R0805
Changed lines of the file:
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@@
 <?xml version="1.0" encoding="utf-8"?>
 <!DOCTYPE eagle SYSTEM "eagle.dtd">
-<eagle version="8.4.2">
+<eagle version="8.4.1">
 <drawing>
 <settings>
@@
 <part name="FCC_1" library="ETHERNET-3" deviceset="ETHERNET" device=""/>
 <part name="FCC_2" library="ETHERNET-3" deviceset="ETHERNET" device=""/>
-<part name="R4" library="Resistor" deviceset="R-US_" device="R0805" value="775 (0.1%)"/>
-<part name="R5" library="Resistor" deviceset="R-US_" device="R0805" value="10.5k (0.1%)"/>
-<part name="R6" library="Resistor" deviceset="R-US_" device="R0805" value="10.5k (0.1%)"/>
-<part name="R7" library="Resistor" deviceset="R-US_" device="R0805" value="775 (0.1%)"/>
+<part name="R4" library="resistor" library_urn="urn:adsk.eagle:library:348" deviceset="R-US_" device="R0805" package3d_urn="urn:adsk.eagle:package:26059/1" value="775 (0.1%)"/>
+<part name="R5" library="resistor" library_urn="urn:adsk.eagle:library:348" deviceset="R-US_" device="R0805" package3d_urn="urn:adsk.eagle:package:26059/1" value="10.5k (0.1%)"/>
+<part name="R6" library="resistor" library_urn="urn:adsk.eagle:library:348" deviceset="R-US_" device="R0805" package3d_urn="urn:adsk.eagle:package:26059/1" value="10.5k (0.1%)"/>
+<part name="R7" library="resistor" library_urn="urn:adsk.eagle:library:348" deviceset="R-US_" device="R0805" package3d_urn="urn:adsk.eagle:package:26059/1" value="775 (0.1%)"/>
 <part name="U$22" library="Relay_CPC1907B" deviceset="RELAY-CPC1907B" device=""/>
 <part name="FC.POS" library="Connector 732-3204" deviceset="732-3204-ND_CONNECTOR" device=""/>
@@
 <part name="C3" library="SparkFun-Passives" deviceset="CAP" device="0603-CAP"/>
 <part name="CAP.POS" library="Connector 732-3204" deviceset="732-3204-ND_CONNECTOR" device=""/>
-<part name="R2" library="Resistor" deviceset="R-US_" device="R0805" value="775 (0.1%)"/>
-<part name="R8" library="Resistor" deviceset="R-US_" device="R0805" value="10.5k (0.1%)"/>
+<part name="R2" library="resistor" library_urn="urn:adsk.eagle:library:348" deviceset="R-US_" device="R0805" package3d_urn="urn:adsk.eagle:package:26059/1" value="775 (0.1%)"/>
+<part name="R8" library="resistor" library_urn="urn:adsk.eagle:library:348" deviceset="R-US_" device="R0805" package3d_urn="urn:adsk.eagle:package:26059/1" value="10.5k (0.1%)"/>
 <part name="D1" library="Diode - APT60S20SG" deviceset="APT60S20SG" device=""/>
 <part name="U$13" library="Relay 255-5246-ND" deviceset="255-5246-ND" device=""/>
@@
 <part name="U$16" library="TVS Diode Through-Hole" deviceset="P6KE15A-E3/54GICT-ND_TVS_DIODE" device=""/>
 <part name="S1" library="SparkFun-Electromechanical" deviceset="SWITCH-SPDT" device="PTH"/>
-<part name="R14" library="Resistor" deviceset="R-US_" device="R0805" value="1.5k (0.1%)"/>
+<part name="R14" library="resistor" library_urn="urn:adsk.eagle:library:348" deviceset="R-US_" device="R0805" package3d_urn="urn:adsk.eagle:package:26059/1" value="1.5k (0.1%)"/>
 <part name="S2" library="SparkFun-Electromechanical" deviceset="SWITCH-SPDT" device="PTH"/>
 <part name="S3" library="SparkFun-Electromechanical" deviceset="SWITCH-SPDT" device="PTH"/>
-<part name="R15" library="Resistor" deviceset="R-US_" device="R0805" value="1.5k (0.1%)"/>
-<part name="R16" library="Resistor" deviceset="R-US_" device="R0805" value="1.5k (0.1%)"/>
+<part name="R15" library="resistor" library_urn="urn:adsk.eagle:library:348" deviceset="R-US_" device="R0805" package3d_urn="urn:adsk.eagle:package:26059/1" value="1.5k (0.1%)"/>
+<part name="R16" library="resistor" library_urn="urn:adsk.eagle:library:348" deviceset="R-US_" device="R0805" package3d_urn="urn:adsk.eagle:package:26059/1" value="1.5k (0.1%)"/>
 </parts>
 <sheets>
@@
 which will not be processed correctly with this version.
 </note>
+<note version="8.2" severity="warning">
+Since Version 8.2, EAGLE supports online libraries. The ids
+of those online libraries will not be understood (or retained)
+with this version.
+</note>
+<note version="8.3" severity="warning">
+Since Version 8.3, EAGLE supports URNs for individual library
+assets (packages, symbols, and devices). The URNs of those assets
+will not be understood (or retained) with this version.
+</note>
+<note version="8.3" severity="warning">
+Since Version 8.3, EAGLE supports the association of 3D packages
+with devices in libraries, schematics, and board files. Those 3D
+packages will not be understood (or retained) with this version.
+</note>
 </compatibility>

Commit message: Added Labels to Ethernet connectors
Parts:
- U$19: value 5555140-6 -> TO POWERBOARD
- renumbered FCC_1 to RELAY1, FCC_2 to RELAY2
Changed lines of the file:
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@@
 </classes>
 <parts>
-<part name="FCC_1" library="ETHERNET-3" deviceset="ETHERNET" device=""/>
-<part name="FCC_2" library="ETHERNET-3" deviceset="ETHERNET" device=""/>
+<part name="RELAY1" library="ETHERNET-3" deviceset="ETHERNET" device=""/>
+<part name="RELAY2" library="ETHERNET-3" deviceset="ETHERNET" device=""/>
 <part name="R4" library="resistor" library_urn="urn:adsk.eagle:library:348" deviceset="R-US_" device="R0805" package3d_urn="urn:adsk.eagle:package:26059/1" value="775 (0.1%)"/>
 <part name="R5" library="resistor" library_urn="urn:adsk.eagle:library:348" deviceset="R-US_" device="R0805" package3d_urn="urn:adsk.eagle:package:26059/1" value="10.5k (0.1%)"/>
@@
 <part name="MOTOR.GROUND" library="Connector 732-3204" deviceset="732-3204-ND_CONNECTOR" device=""/>
 <part name="CAP.GND" library="Connector 732-3204" deviceset="732-3204-ND_CONNECTOR" device=""/>
-<part name="U$19" library="5555140-6 RJ11" deviceset="5555140-6" device=""/>
+<part name="U$19" library="5555140-6 RJ11" deviceset="5555140-6" device="" value="TO POWERBOARD"/>
 <part name="START.RELAY1" library="VCF4-1000" deviceset="VCF4-1000" device=""/>
 <part name="U$11" library="DMP3056L-7" deviceset="DMP3056L-7" device="DMP3056L-7"/>
@@
 </plain>
 <instances>
-<instance part="FCC_1" gate="G$1" x="172.72" y="17.78"/>
-<instance part="FCC_2" gate="G$1" x="172.72" y="-38.1"/>
+<instance part="RELAY1" gate="G$1" x="172.72" y="17.78"/>
+<instance part="RELAY2" gate="G$1" x="172.72" y="-38.1"/>
 <instance part="R4" gate="G$1" x="104.14" y="78.74"/>
 <instance part="R5" gate="G$1" x="66.04" y="73.66"/>
@@
 </segment>
 <segment>
-<pinref part="FCC_1" gate="G$1" pin="1"/>
+<pinref part="RELAY1" gate="G$1" pin="1"/>
 <wire x1="167.64" y1="33.02" x2="162.56" y2="33.02" width="0.1524" layer="91"/>
 <label x="154.94" y="33.02" size="1.778" layer="95"/>
 </segment>
 <segment>
-<pinref part="FCC_2" gate="G$1" pin="7"/>
+<pinref part="RELAY2" gate="G$1" pin="7"/>
 <wire x1="162.56" y1="-38.1" x2="167.64" y2="-38.1" width="0.1524" layer="91"/>
 <label x="154.94" y="-38.1" size="1.778" layer="95"/>
@@
 </segment>
 <segment>
-<pinref part="FCC_2" gate="G$1" pin="8"/>
+<pinref part="RELAY2" gate="G$1" pin="8"/>
 <wire x1="167.64" y1="-40.64" x2="162.56" y2="-40.64" width="0.1524" layer="91"/>
 <label x="154.94" y="-40.64" size="1.778" layer="95"/>
@@
 </segment>
 <segment>
-<pinref part="FCC_2" gate="G$1" pin="4"/>
+<pinref part="RELAY2" gate="G$1" pin="4"/>
 <wire x1="162.56" y1="-30.48" x2="167.64" y2="-30.48" width="0.1524" layer="91"/>
 <label x="154.94" y="-30.48" size="1.778" layer="95"/>
@@
 </segment>
 <segment>
-<pinref part="FCC_2" gate="G$1" pin="1"/>
+<pinref part="RELAY2" gate="G$1" pin="1"/>
 <wire x1="162.56" y1="-22.86" x2="167.64" y2="-22.86" width="0.1524" layer="91"/>
 <label x="154.94" y="-22.86" size="1.778" layer="95"/>
@@
 </segment>
 <segment>
-<pinref part="FCC_1" gate="G$1" pin="2"/>
+<pinref part="RELAY1" gate="G$1" pin="2"/>
 <wire x1="162.56" y1="30.48" x2="167.64" y2="30.48" width="0.1524" layer="91"/>
 <label x="154.94" y="30.48" size="1.778" layer="95"/>
@@
 </segment>
 <segment>
-<pinref part="FCC_2" gate="G$1" pin="5"/>
+<pinref part="RELAY2" gate="G$1" pin="5"/>
 <wire x1="162.56" y1="-33.02" x2="167.64" y2="-33.02" width="0.1524" layer="91"/>
 <label x="154.94" y="-33.02" size="1.778" layer="95"/>
@@
 </segment>
 <segment>
-<pinref part="FCC_2" gate="G$1" pin="6"/>
+<pinref part="RELAY2" gate="G$1" pin="6"/>
 <wire x1="162.56" y1="-35.56" x2="167.64" y2="-35.56" width="0.1524" layer="91"/>
 <label x="154.94" y="-35.56" size="1.778" layer="95"/>
@@
 <net name="CAP_R" class="0">
 <segment>
-<pinref part="FCC_1" gate="G$1" pin="3"/>
+<pinref part="RELAY1" gate="G$1" pin="3"/>
 <wire x1="162.56" y1="27.94" x2="167.64" y2="27.94" width="0.1524" layer="91"/>
 <label x="154.94" y="27.94" size="1.778" layer="95"/>
@@
 <net name="MOTOR_R" class="0">
 <segment>
-<pinref part="FCC_1" gate="G$1" pin="4"/>
+<pinref part="RELAY1" gate="G$1" pin="4"/>
 <wire x1="162.56" y1="25.4" x2="167.64" y2="25.4" width="0.1524" layer="91"/>
 <label x="154.94" y="25.4" size="1.778" layer="95"/>
@@
 <net name="START_R" class="0">
 <segment>
-<pinref part="FCC_1" gate="G$1" pin="5"/>
+<pinref part="RELAY1" gate="G$1" pin="5"/>
 <wire x1="162.56" y1="22.86" x2="167.64" y2="22.86" width="0.1524" layer="91"/>
 <label x="154.94" y="22.86" size="1.778" layer="95"/>
@@
 <net name="CHARGE_R" class="0">
 <segment>
-<pinref part="FCC_1" gate="G$1" pin="6"/>
+<pinref part="RELAY1" gate="G$1" pin="6"/>
 <wire x1="162.56" y1="20.32" x2="167.64" y2="20.32" width="0.1524" layer="91"/>
 <label x="154.94" y="20.32" size="1.778" layer="95"/>
@@
 <net name="ISO_GND" class="0">
 <segment>
-<pinref part="FCC_1" gate="G$1" pin="7"/>
+<pinref part="RELAY1" gate="G$1" pin="7"/>
 <wire x1="162.56" y1="17.78" x2="167.64" y2="17.78" width="0.1524" layer="91"/>
 <label x="154.94" y="17.78" size="1.778" layer="95"/>
 </segment>
 <segment>
-<pinref part="FCC_1" gate="G$1" pin="8"/>
+<pinref part="RELAY1" gate="G$1" pin="8"/>
 <wire x1="162.56" y1="15.24" x2="167.64" y2="15.24" width="0.1524" layer="91"/>
 <label x="154.94" y="15.24" size="1.778" layer="95"/>
 </segment>
 <segment>
-<pinref part="FCC_2" gate="G$1" pin="SHD1"/>
+<pinref part="RELAY2" gate="G$1" pin="SHD1"/>
 <wire x1="167.64" y1="-53.34" x2="162.56" y2="-53.34" width="0.1524" layer="91"/>
 <label x="154.94" y="-53.34" size="1.778" layer="95"/>
 </segment>
 <segment>
-<pinref part="FCC_2" gate="G$1" pin="SHD2"/>
+<pinref part="RELAY2" gate="G$1" pin="SHD2"/>
 <wire x1="162.56" y1="-55.88" x2="167.64" y2="-55.88" width="0.1524" layer="91"/>
 <label x="154.94" y="-55.88" size="1.778" layer="95"/>
 </segment>
 <segment>
-<pinref part="FCC_1" gate="G$1" pin="SHD1"/>
+<pinref part="RELAY1" gate="G$1" pin="SHD1"/>
 <wire x1="167.64" y1="2.54" x2="162.56" y2="2.54" width="0.1524" layer="91"/>
 <label x="154.94" y="2.54" size="1.778" layer="95"/>
 </segment>
 <segment>
-<pinref part="FCC_1" gate="G$1" pin="SHD2"/>
+<pinref part="RELAY1" gate="G$1" pin="SHD2"/>
 <wire x1="167.64" y1="0" x2="162.56" y2="0" width="0.1524" layer="91"/>
 <label x="154.94" y="0" size="1.778" layer="95"/>
@@
 <net name="CAP_VOLT" class="0">
 <segment>
-<pinref part="FCC_2" gate="G$1" pin="2"/>
+<pinref part="RELAY2" gate="G$1" pin="2"/>
 <wire x1="162.56" y1="-25.4" x2="167.64" y2="-25.4" width="0.1524" layer="91"/>
 <label x="154.94" y="-25.4" size="1.778" layer="95"/>
@@
 <net name="MOTOR_VOLT" class="0">
 <segment>
-<pinref part="FCC_2" gate="G$1" pin="3"/>
+<pinref part="RELAY2" gate="G$1" pin="3"/>
 <wire x1="162.56" y1="-27.94" x2="167.64" y2="-27.94" width="0.1524" layer="91"/>
 <label x="154.94" y="-27.94" size="1.778" layer="95"/>
