File: Relay_Board_V3.2.sch (EAGLE design)
At the start: 59 parts

Commit message: Added RJ-11
Parts:
- added U$10, U$17: 5555140-6, 5555140-6 RJ11:5555140-6
Connections:
- net 5V: now also U$17.2, U$17.5
- net AUX.12: now also U$10.3, U$10.4
- net CAP_CURR: now also FCC_2.6; no longer FCC_2.5
- net CAP_VOLT: now also FCC_2.3; no longer FCC_2.2
- net FC.12: now also U$17.3, U$17.4
- net GND: now also U$10.1, U$10.6, U$10.SH1, U$10.SH2, U$17.1, U$17.6, U$17.SH1, U$17.SH2
- net MOTOR_CURR: now also FCC_2.5; no longer FCC_2.6
- net MOTOR_VOLT: now also FCC_2.2; no longer FCC_2.3
Changed lines of the file:
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@@
 <part name="R15" library="Resistor" deviceset="R-US_" device="R0805" value="1.5k (0.1%)"/>
 <part name="R16" library="Resistor" deviceset="R-US_" device="R0805" value="1.5k (0.1%)"/>
+<part name="U$10" library="5555140-6 RJ11" deviceset="5555140-6" device=""/>
+<part name="U$17" library="5555140-6 RJ11" deviceset="5555140-6" device=""/>
 </parts>
 <sheets>
@@
 <instance part="R15" gate="G$1" x="104.14" y="88.9"/>
 <instance part="R16" gate="G$1" x="104.14" y="48.26"/>
+<instance part="U$10" gate="G$1" x="218.44" y="81.28"/>
+<instance part="U$17" gate="G$1" x="218.44" y="33.02"/>
 </instances>
 <busses>
@@
 <wire x1="162.56" y1="-38.1" x2="167.64" y2="-38.1" width="0.1524" layer="91"/>
 <label x="154.94" y="-38.1" size="1.778" layer="95"/>
+</segment>
+<segment>
+<pinref part="U$17" gate="G$1" pin="2"/>
+<wire x1="210.82" y1="40.64" x2="205.74" y2="40.64" width="0.1524" layer="91"/>
+<label x="203.2" y="40.64" size="1.778" layer="95"/>
+</segment>
+<segment>
+<pinref part="U$17" gate="G$1" pin="5"/>
+<wire x1="210.82" y1="25.4" x2="205.74" y2="25.4" width="0.1524" layer="91"/>
+<label x="203.2" y="25.4" size="1.778" layer="95"/>
 </segment>
 </net>
@@
 <label x="114.3" y="53.34" size="1.778" layer="95"/>
 </segment>
+<segment>
+<pinref part="U$10" gate="G$1" pin="1"/>
+<wire x1="210.82" y1="93.98" x2="205.74" y2="93.98" width="0.1524" layer="91"/>
+<label x="203.2" y="93.98" size="1.778" layer="95"/>
+</segment>
+<segment>
+<pinref part="U$10" gate="G$1" pin="6"/>
+<wire x1="210.82" y1="68.58" x2="205.74" y2="68.58" width="0.1524" layer="91"/>
+<label x="203.2" y="68.58" size="1.778" layer="95"/>
+</segment>
+<segment>
+<pinref part="U$10" gate="G$1" pin="SH1"/>
+<wire x1="210.82" y1="63.5" x2="205.74" y2="63.5" width="0.1524" layer="91"/>
+<label x="203.2" y="63.5" size="1.778" layer="95"/>
+</segment>
+<segment>
+<pinref part="U$10" gate="G$1" pin="SH2"/>
+<wire x1="210.82" y1="58.42" x2="205.74" y2="58.42" width="0.1524" layer="91"/>
+<label x="203.2" y="58.42" size="1.778" layer="95"/>
+</segment>
+<segment>
+<pinref part="U$17" gate="G$1" pin="1"/>
+<wire x1="210.82" y1="45.72" x2="205.74" y2="45.72" width="0.1524" layer="91"/>
+<label x="203.2" y="45.72" size="1.778" layer="95"/>
+</segment>
+<segment>
+<pinref part="U$17" gate="G$1" pin="6"/>
+<wire x1="210.82" y1="20.32" x2="205.74" y2="20.32" width="0.1524" layer="91"/>
+<label x="203.2" y="20.32" size="1.778" layer="95"/>
+</segment>
+<segment>
+<pinref part="U$17" gate="G$1" pin="SH1"/>
+<wire x1="210.82" y1="15.24" x2="205.74" y2="15.24" width="0.1524" layer="91"/>
+<label x="203.2" y="15.24" size="1.778" layer="95"/>
+</segment>
+<segment>
+<pinref part="U$17" gate="G$1" pin="SH2"/>
+<wire x1="210.82" y1="10.16" x2="205.74" y2="10.16" width="0.1524" layer="91"/>
+<label x="203.2" y="10.16" size="1.778" layer="95"/>
+</segment>
 </net>
 <net name="FC_CURR" class="0">
@@
 </segment>
 <segment>
-<pinref part="FCC_2" gate="G$1" pin="5"/>
-<wire x1="162.56" y1="-33.02" x2="167.64" y2="-33.02" width="0.1524" layer="91"/>
-<label x="154.94" y="-33.02" size="1.778" layer="95"/>
+<pinref part="FCC_2" gate="G$1" pin="6"/>
+<wire x1="167.64" y1="-35.56" x2="162.56" y2="-35.56" width="0.1524" layer="91"/>
+<label x="154.94" y="-35.56" size="1.778" layer="95"/>
 </segment>
 </net>
@@
 </segment>
 <segment>
-<pinref part="FCC_2" gate="G$1" pin="6"/>
-<wire x1="162.56" y1="-35.56" x2="167.64" y2="-35.56" width="0.1524" layer="91"/>
-<label x="154.94" y="-35.56" size="1.778" layer="95"/>
+<pinref part="FCC_2" gate="G$1" pin="5"/>
+<wire x1="167.64" y1="-33.02" x2="162.56" y2="-33.02" width="0.1524" layer="91"/>
+<label x="154.94" y="-33.02" size="1.778" layer="95"/>
 </segment>
 </net>
@@
 <net name="CAP_VOLT" class="0">
 <segment>
-<pinref part="FCC_2" gate="G$1" pin="2"/>
-<wire x1="162.56" y1="-25.4" x2="167.64" y2="-25.4" width="0.1524" layer="91"/>
-<label x="154.94" y="-25.4" size="1.778" layer="95"/>
-</segment>
-<segment>
 <pinref part="R5" gate="G$1" pin="2"/>
 <wire x1="91.44" y1="73.66" x2="71.12" y2="73.66" width="0.1524" layer="91"/>
@@
 <pinref part="S1" gate="1" pin="P"/>
 </segment>
+<segment>
+<pinref part="FCC_2" gate="G$1" pin="3"/>
+<wire x1="167.64" y1="-27.94" x2="162.56" y2="-27.94" width="0.1524" layer="91"/>
+<label x="154.94" y="-27.94" size="1.778" layer="95"/>
+</segment>
 </net>
 <net name="MOTOR_VOLT" class="0">
-<segment>
-<pinref part="FCC_2" gate="G$1" pin="3"/>
-<wire x1="162.56" y1="-27.94" x2="167.64" y2="-27.94" width="0.1524" layer="91"/>
-<label x="154.94" y="-27.94" size="1.778" layer="95"/>
-</segment>
 <segment>
 <pinref part="R8" gate="G$1" pin="2"/>
@@
 <pinref part="S3" gate="1" pin="P"/>
 </segment>
+<segment>
+<pinref part="FCC_2" gate="G$1" pin="2"/>
+<wire x1="167.64" y1="-25.4" x2="162.56" y2="-25.4" width="0.1524" layer="91"/>
+<label x="154.94" y="-25.4" size="1.778" layer="95"/>
+</segment>
 </net>
 <net name="AUX.12" class="0">
@@
 <label x="132.08" y="63.5" size="1.778" layer="95" rot="R90"/>
 </segment>
+<segment>
+<pinref part="U$10" gate="G$1" pin="3"/>
+<wire x1="210.82" y1="83.82" x2="205.74" y2="83.82" width="0.1524" layer="91"/>
+<label x="203.2" y="83.82" size="1.778" layer="95"/>
+</segment>
+<segment>
+<pinref part="U$10" gate="G$1" pin="4"/>
+<wire x1="210.82" y1="78.74" x2="205.74" y2="78.74" width="0.1524" layer="91"/>
+<label x="203.2" y="78.74" size="1.778" layer="95"/>
+</segment>
 </net>
 <net name="FC.12" class="0">
@@
 <label x="144.78" y="63.5" size="1.778" layer="95" rot="R90"/>
 </segment>
-</net>
+<segment>
+<pinref part="U$17" gate="G$1" pin="3"/>
+<wire x1="210.82" y1="35.56" x2="205.74" y2="35.56" width="0.1524" layer="91"/>
+<label x="203.2" y="35.56" size="1.778" layer="95"/>
+</segment>
+<segment>
+<pinref part="U$17" gate="G$1" pin="4"/>
+<wire x1="210.82" y1="30.48" x2="205.74" y2="30.48" width="0.1524" layer="91"/>
+<label x="203.2" y="30.48" size="1.778" layer="95"/>
+</segment>
+</net>
