File: Relay_Board_V3.3.brd (EAGLE design)
At the start: 160 x 100 mm, 65 parts

Commit message: Schematic Fix
Parts:
- C1, C2, C3: value (none) -> 0.1u
Changed lines of the file:
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@@
 <element name="CAP.POS2" library="Connector 732-3204" package="732-3204-ND" value="732-3204-ND_CONNECTOR" x="88" y="92"/>
 <element name="U$7" library="ACS770 Current Sensor" package="ACS770LCB_CURRENTSENSOR" value="ACS770LCB_CURRENTSENSOR" x="31" y="68" rot="R90"/>
-<element name="C1" library="SparkFun-Passives" package="0603-CAP" value="" x="112.5" y="45.5" rot="MR0"/>
+<element name="C1" library="SparkFun-Passives" package="0603-CAP" value="0.1u" x="112.5" y="45.5" rot="MR0"/>
 <element name="U$8" library="ACS770 Current Sensor" package="ACS770LCB_CURRENTSENSOR" value="ACS770LCB_CURRENTSENSOR" x="111.5" y="27" rot="R180"/>
 <element name="U$9" library="ACS770 Current Sensor" package="ACS770LCB_CURRENTSENSOR" value="ACS770LCB_CURRENTSENSOR" x="61" y="52"/>
-<element name="C2" library="SparkFun-Passives" package="0603-CAP" value="" x="49.5" y="67" rot="MR90"/>
-<element name="C3" library="SparkFun-Passives" package="0603-CAP" value="" x="60" y="33" rot="MR180"/>
+<element name="C2" library="SparkFun-Passives" package="0603-CAP" value="0.1u" x="49.5" y="67" rot="MR90"/>
+<element name="C3" library="SparkFun-Passives" package="0603-CAP" value="0.1u" x="60" y="33" rot="MR180"/>
 <element name="CAP.POS" library="Connector 732-3204" package="732-3204-ND" value="732-3204-ND_CONNECTOR" x="152.5" y="42"/>
 <element name="R2" library="Resistor" package="R0805" value="775 (0.1%)" x="72" y="59.5" rot="MR270"/>
