File: Relay_Board_V3.3.sch (EAGLE design)
At the start: 61 parts

Commit message: Schematic Fix
Parts:
- C1, C2, C3: value (none) -> 0.1u
Changed lines of the file:
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@@
 <part name="CAP.POS2" library="Connector 732-3204" deviceset="732-3204-ND_CONNECTOR" device=""/>
 <part name="U$7" library="ACS770 Current Sensor" deviceset="ACS770LCB_CURRENTSENSOR" device=""/>
-<part name="C1" library="SparkFun-Passives" deviceset="CAP" device="0603-CAP"/>
+<part name="C1" library="SparkFun-Passives" deviceset="CAP" device="0603-CAP" value="0.1u"/>
 <part name="U$8" library="ACS770 Current Sensor" deviceset="ACS770LCB_CURRENTSENSOR" device=""/>
 <part name="U$9" library="ACS770 Current Sensor" deviceset="ACS770LCB_CURRENTSENSOR" device=""/>
-<part name="C2" library="SparkFun-Passives" deviceset="CAP" device="0603-CAP"/>
-<part name="C3" library="SparkFun-Passives" deviceset="CAP" device="0603-CAP"/>
+<part name="C2" library="SparkFun-Passives" deviceset="CAP" device="0603-CAP" value="0.1u"/>
+<part name="C3" library="SparkFun-Passives" deviceset="CAP" device="0603-CAP" value="0.1u"/>
 <part name="CAP.POS" library="Connector 732-3204" deviceset="732-3204-ND_CONNECTOR" device=""/>
 <part name="R2" library="Resistor" deviceset="R-US_" device="R0805" value="775 (0.1%)"/>
@@
 <wire x1="-121.92" y1="-76.2" x2="30.48" y2="-76.2" width="0.1524" layer="94"/>
 <wire x1="30.48" y1="-76.2" x2="139.7" y2="-76.2" width="0.1524" layer="94"/>
-<wire x1="139.7" y1="-76.2" x2="190.5" y2="-76.2" width="0.1524" layer="94"/>
-<wire x1="190.5" y1="-76.2" x2="190.5" y2="127" width="0.1524" layer="94"/>
-<wire x1="190.5" y1="127" x2="121.92" y2="127" width="0.1524" layer="94"/>
+<wire x1="139.7" y1="-76.2" x2="231.14" y2="-76.2" width="0.1524" layer="94"/>
+<wire x1="231.14" y1="-76.2" x2="231.14" y2="127" width="0.1524" layer="94"/>
+<wire x1="231.14" y1="127" x2="121.92" y2="127" width="0.1524" layer="94"/>
 <wire x1="121.92" y1="127" x2="30.48" y2="127" width="0.1524" layer="94"/>
 <wire x1="30.48" y1="127" x2="-121.92" y2="127" width="0.1524" layer="94"/>
@@
 <wire x1="-12.7" y1="5.08" x2="-12.7" y2="10.16" width="0.1524" layer="91"/>
 <label x="-12.7" y="10.16" size="1.778" layer="95"/>
+<junction x="-22.86" y="5.08"/>
 </segment>
 <segment>
@@
 <wire x1="111.76" y1="73.66" x2="114.3" y2="73.66" width="0.1524" layer="91"/>
 <label x="114.3" y="73.66" size="1.778" layer="95"/>
+<junction x="111.76" y="73.66"/>
 </segment>
 <segment>
@@
 <wire x1="111.76" y1="93.98" x2="114.3" y2="93.98" width="0.1524" layer="91"/>
 <label x="114.3" y="93.98" size="1.778" layer="95"/>
+<junction x="111.76" y="93.98"/>
 </segment>
 <segment>
@@
 <wire x1="111.76" y1="53.34" x2="114.3" y2="53.34" width="0.1524" layer="91"/>
 <label x="114.3" y="53.34" size="1.778" layer="95"/>
+<junction x="111.76" y="53.34"/>
 </segment>
 <segment>
@@
 <label x="-20.32" y="38.1" size="1.778" layer="95"/>
 <pinref part="D1" gate="G$1" pin="(-)"/>
+<junction x="-33.02" y="38.1"/>
 </segment>
 <segment>
@@
 <wire x1="-78.74" y1="-83.82" x2="-78.74" y2="-91.44" width="0.1524" layer="91"/>
 <wire x1="-78.74" y1="-91.44" x2="-60.96" y2="-91.44" width="0.1524" layer="91"/>
+<junction x="-60.96" y="-91.44"/>
 </segment>
 <segment>
@@
 <pinref part="START.RELAY2" gate="G$1" pin="85"/>
 <wire x1="-60.96" y1="22.86" x2="-60.96" y2="17.78" width="0.1524" layer="91"/>
+<junction x="-60.96" y="17.78"/>
 </segment>
 <segment>
@@
 <pinref part="U$14" gate="G$1" pin="(-)"/>
 <wire x1="121.92" y1="-83.82" x2="119.38" y2="-83.82" width="0.1524" layer="91"/>
+<junction x="119.38" y="-91.44"/>
 </segment>
 <segment>
@@
 <pinref part="U$13" gate="G$1" pin="(-)"/>
 <wire x1="121.92" y1="22.86" x2="119.38" y2="22.86" width="0.1524" layer="91"/>
+<junction x="119.38" y="15.24"/>
 </segment>
 </net>
@@
 <wire x1="-78.74" y1="-63.5" x2="-78.74" y2="-48.26" width="0.1524" layer="91"/>
 <wire x1="-78.74" y1="-48.26" x2="-60.96" y2="-48.26" width="0.1524" layer="91"/>
+<junction x="-60.96" y="-48.26"/>
 </segment>
 </net>
@@
 <pinref part="START.RELAY2" gate="G$1" pin="86"/>
 <wire x1="-60.96" y1="60.96" x2="-60.96" y2="53.34" width="0.1524" layer="91"/>
+<junction x="-60.96" y="60.96"/>
 </segment>
 </net>
@@
 <pinref part="U$14" gate="G$1" pin="(+)"/>
 <wire x1="121.92" y1="-66.04" x2="119.38" y2="-66.04" width="0.1524" layer="91"/>
+<junction x="119.38" y="-48.26"/>
 </segment>
 </net>
@@
 <pinref part="U$13" gate="G$1" pin="(+)"/>
 <wire x1="121.92" y1="40.64" x2="119.38" y2="40.64" width="0.1524" layer="91"/>
-</segment>
-</net>
+<junction x="119.38" y="58.42"/>
+</segment>
+</net>
